File: kicad/bms-c1.kicad_pcb (KiCad board)
At the start: 4 copper layers, 135 x 70 mm, 209 parts, among them J1 MicroFit 2x12, J2 B4B-PH-SM4, J3 USB_C_Receptacle_USB2.0, J4 B3B-PH-SM4, J5 B2B-PH-SM4, J6 B4B-PH-SM4, P1 CONN_01X01, P2 CONN_01X01, P3 CONN_01X01, P4 CONN_01X01, P5 CONN_01X01, Q1 DMN10H220LE, Q10 BSS84, Q11 BSS123N, Q12 ZXMP10A17GTA, Q2 IPT012N08N5, Q3 IPT012N08N5, Q4 IPT012N08N5, Q5 IPT012N08N5, Q6 IPT012N08N5, Q7 IPT012N08N5, Q8 IPT012N08N5, Q9 IPT012N08N5, U1 SN65HVD230, U2 SN65HVD75, U3 LMR38010, U4 BQ76952, U5 ESP32-C3-MINI-1

Commit message: fix: Replace REF** in WEEE Logo with meaningfull name
Parts:
- renumbered REF** to LOGO3
Changed lines of the file:
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@@
     (tags "Logo WEEE")
     (attr exclude_from_pos_files exclude_from_bom)
-    (fp_text reference "REF**" (at 0 0) (layer "F.SilkS") hide
+    (fp_text reference "LOGO3" (at 0 0) (layer "F.SilkS") hide
         (effects (font (size 1 1) (thickness 0.15)))
     )
