File: kicad/esp32-c3.kicad_sch (KiCad schematic)
At the start: 19 parts, among them U1 SN65HVD230, U2 SN65HVD75, U5 ESP32-C3-MINI-1

Commit message: fix: Field conflict remarks
kibot throws following warning:
WARNING:(W004) Field conflict: (C30,C47) [remarks] : 'min. 25V, X5R' <- 'min. 10V, X5R' (in C47) (kibot - bom.py:299)

So correct all CL10A105KA8NNNC parts.
Parts:
- C47: Remarks min. 10V, X5R -> min. 25V, X5R
Changed lines of the file:
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@@
       (effects (font (size 1.27 1.27)) hide)
     )
-    (property "Remarks" "min. 10V, X5R" (at 48.26 68.58 0)
+    (property "Remarks" "min. 25V, X5R" (at 48.26 68.58 0)
       (effects (font (size 1.27 1.27)) hide)
     )
