File: kicad/power-part.kicad_sch (KiCad schematic)
At the start: 53 parts, among them Q10 BSS84, Q11 BSS123N, Q12 ZXMP10A17GTA, Q2 IPT012N08N5, Q3 IPT012N08N5, Q4 IPT012N08N5, Q5 IPT012N08N5, Q6 IPT012N08N5, Q7 IPT012N08N5, Q8 IPT012N08N5, Q9 IPT012N08N5

Commit message: fix: Field Remarks of component Q5 contains extra spaces
kibot throws following warnings:
WARNING:(W037) Field Remarks of component Q5 (Q_NMOS_GSD IPT012N08N5) contains extra spaces: `Alternative: Huayi HYG012N08NS1TA ` removing them. (kibot - v5_sch.py:1057)
WARNING:(W037) Field Remarks of component Q3 (Q_NMOS_GSD IPT012N08N5) contains extra spaces: `Alternative: Huayi HYG012N08NS1TA ` removing them. (kibot - v5_sch.py:1057)
WARNING:(W037) Field Remarks of component Q4 (Q_NMOS_GSD IPT012N08N5) contains extra spaces: `Alternative: Huayi HYG012N08NS1TA ` removing them. (kibot - v5_sch.py:1057)
WARNING:(W037) Field Remarks of component Q9 (Q_NMOS_GSD IPT012N08N5) contains extra spaces: `Alternative: Huayi HYG012N08NS1TA ` removing them. (kibot - v5_sch.py:1057)
WARNING:(W037) Field Remarks of component Q2 (Q_NMOS_GSD IPT012N08N5) contains extra spaces: `Alternative: Huayi HYG012N08NS1TA ` removing them. (kibot - v5_sch.py:1057)
WARNING:(W037) Field Remarks of component Q6 (Q_NMOS_GSD IPT012N08N5) contains extra spaces: `Alternative: Huayi HYG012N08NS1TA ` removing them. (kibot - v5_sch.py:1057)
WARNING:(W037) Field Remarks of component Q8 (Q_NMOS_GSD IPT012N08N5) contains extra spaces: `Alternative: Huayi HYG012N08NS1TA ` removing them. (kibot - v5_sch.py:1057)
WARNING:(W037) Field Remarks of component Q7 (Q_NMOS_GSD IPT012N08N5) contains extra spaces: `Alternative: Huayi HYG012N08NS1TA ` removing them. (kibot - v5_sch.py:1057)
Parts:
- Q2, Q3, Q4, Q5, Q6, Q7, Q8, Q9: Remarks Alternative: Huayi HYG012N08NS1TA -> Alternative: Huayi HYG012N08NS1TA
Changed lines of the file:
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@@
       (effects (font (size 1.27 1.27)) hide)
     )
-    (property "Remarks" "Alternative: Huayi HYG012N08NS1TA " (at 96.52 119.38 0)
+    (property "Remarks" "Alternative: Huayi HYG012N08NS1TA" (at 96.52 119.38 0)
       (effects (font (size 1.27 1.27)) hide)
     )
@@
       (effects (font (size 1.27 1.27)) hide)
     )
-    (property "Remarks" "Alternative: Huayi HYG012N08NS1TA " (at 96.52 83.82 0)
+    (property "Remarks" "Alternative: Huayi HYG012N08NS1TA" (at 96.52 83.82 0)
       (effects (font (size 1.27 1.27)) hide)
     )
@@
       (effects (font (size 1.27 1.27)) hide)
     )
-    (property "Remarks" "Alternative: Huayi HYG012N08NS1TA " (at 96.52 101.6 0)
+    (property "Remarks" "Alternative: Huayi HYG012N08NS1TA" (at 96.52 101.6 0)
       (effects (font (size 1.27 1.27)) hide)
     )
@@
       (effects (font (size 1.27 1.27)) hide)
     )
-    (property "Remarks" "Alternative: Huayi HYG012N08NS1TA " (at 129.54 119.38 0)
+    (property "Remarks" "Alternative: Huayi HYG012N08NS1TA" (at 129.54 119.38 0)
       (effects (font (size 1.27 1.27)) hide)
     )
@@
       (effects (font (size 1.27 1.27)) hide)
     )
-    (property "Remarks" "Alternative: Huayi HYG012N08NS1TA " (at 96.52 66.04 0)
+    (property "Remarks" "Alternative: Huayi HYG012N08NS1TA" (at 96.52 66.04 0)
       (effects (font (size 1.27 1.27)) hide)
     )
@@
       (effects (font (size 1.27 1.27)) hide)
     )
-    (property "Remarks" "Alternative: Huayi HYG012N08NS1TA " (at 129.54 66.04 0)
+    (property "Remarks" "Alternative: Huayi HYG012N08NS1TA" (at 129.54 66.04 0)
       (effects (font (size 1.27 1.27)) hide)
     )
@@
       (effects (font (size 1.27 1.27)) hide)
     )
-    (property "Remarks" "Alternative: Huayi HYG012N08NS1TA " (at 129.54 101.6 0)
+    (property "Remarks" "Alternative: Huayi HYG012N08NS1TA" (at 129.54 101.6 0)
       (effects (font (size 1.27 1.27)) hide)
     )
@@
       (effects (font (size 1.27 1.27)) hide)
     )
-    (property "Remarks" "Alternative: Huayi HYG012N08NS1TA " (at 129.54 83.82 0)
-      (effects (font (size 1.27 1.27)) hide)
-    )
+    (property "Remarks" "Alternative: Huayi HYG012N08NS1TA" (at 129.54 83.82 0)
+      (effects (font (size 1.27 1.27)) hide)
+    )
