File: kicad/bms-c1.kicad_sch (KiCad schematic)
At the start: 34 parts, among them J1 MicroFit 2x12, J2 B4B-PH-SM4, J3 USB_C_Receptacle_USB2.0, J4 B3B-PH-SM4, J5 B2B-PH-SM4, J6 B4B-PH-SM4, P1 CONN_01X01, P2 CONN_01X01, P3 CONN_01X01, P4 CONN_01X01, P5 CONN_01X01

Commit message: test for diff
Other:
- note added: "Internal I2C TEST diff"
- note removed: "Internal I2C"
Changed lines of the file:
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@@
     (effects (font (size 2.54 2.54)) (justify left bottom))
   )
-  (text "Internal I2C" (at 30.48 53.34 0)
+  (text "Internal I2C TEST diff" (at 30.48 53.34 0)
     (effects (font (size 2.54 2.54)) (justify left bottom))
   )
