File: kicad/bms-c1.kicad_sch (KiCad schematic)
At the start: 34 parts, among them J1 MicroFit 2x12, J2 B4B-PH-SM4, J3 USB_C_Receptacle_USB2.0, J4 B3B-PH-SM4, J5 B2B-PH-SM4, J6 B4B-PH-SM4, P1 CONN_01X01, P2 CONN_01X01, P3 CONN_01X01, P4 CONN_01X01, P5 CONN_01X01

Commit message: just a test
Other:
- sheet Power Part renamed Power Part (added something)
Changed lines of the file:
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@@
     (stroke (width 0.1524) (type solid))
     (fill (color 0 0 0 0.0000))
-    (property "Sheetname" "Power Part" (at 91.44 42.4684 0)
+    (property "Sheetname" "Power Part (added something)" (at 91.44 42.4684 0)
       (effects (font (size 2.54 2.54)) (justify left bottom))
     )
